Commit message: chore: clean up and minor fixes

File: eagerx_franka/solid/assets/bolt.urdf (robot description, URDF)
Before this commit: robot box, 1 links, 0 joints
Links:
- link baseLink: geometry collision mesh filename=bolt.stl scale=0.01 0.01 0.01; visual mesh filename=bolt.stl scale=0.001 0.001 0.001

File: eagerx_franka/solid/assets/nut.urdf (robot description, URDF)
Before this commit: robot box, 1 links, 0 joints
Links:
- link baseLink: geometry collision mesh filename=nut.stl scale=0.01 0.01 0.01; visual mesh filename=nut.stl scale=0.001 0.001 0.001
